File: mezzanine_round_bond_PCB_new/mezzanine.kicad_pcb (KiCad board)
At the start: 4 copper layers, 16 x 16 mm, 3 parts, among them J101 Conn_02x35_Counter_Clockwise_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, J102 Conn_2Rows-76Pins

Commit message: updates for round-PAD 1108
Other:
- board text added: "70 PIN MEZZANINE 74 PIN PADRING"
- board text added: "wafer.space GF180MCU Run 1"
