File: mezzanine_round_bond_new/mezzanine.kicad_pcb (KiCad board)
At the start: 4 copper layers, 16 x 16 mm, 3 parts, among them J101 Conn_02x35_Counter_Clockwise_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, J102 Conn_2Rows-76Pins

Commit message: update of mezzanine round bond PCB 1118
Connections:
- J102 pad  75: (no net) -> GND
Routing:
- net GND: track 12.8 -> 46.7 mm, vias 3 -> 23
- net (no net): track 3.63 -> 0.00 mm
Other:
- board text removed: "70 PIN MEZZANINE 74 PIN PADRING"
- board text removed: "wafer.space GF180MCU Run 1"
