File: mezzanine_round_bond_new/mezzanine.kicad_sch (KiCad schematic)
At the start: 2 parts, among them J101 Conn_02x35_Counter_Clockwise_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, J102 Conn_2Rows-76Pins

Commit message: update of mezzanine round bond PCB 1118
Changed lines of the file:
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@@
+	(wire
+		(pts
+			(xy 72.39 167.64) (xy 77.47 167.64)
+		)
+		(stroke
+			(width 0)
+			(type default)
+		)
+	)
 	(wire
 		(pts
